Commit message: lively-ik with gripper pass through works but behaves poorly - will need to investigate improvements

File: lik_config/ur3e_new/ur3e_robotiq.urdf (robot description, URDF)
Before this commit: robot ur3e, 20 links, 19 joints
Joints:
- joint gripper_finger1_joint: limit lower=0.0 upper=0.804 effort=1000 velocity=2.0 -> lower=-0.0001 upper=0.0851 effort=100 velocity=1000
- joint gripper_finger2_joint: limit lower=-3.14 upper=3.14 effort=1000 velocity=100.0 -> lower=-0.0001 upper=0.0851 effort=100 velocity=1000
